File: doc/boards/pixelix/v2.0/Pixelix.kicad_sch (KiCad schematic)
At the start: 24 parts

Commit message: Board v2.0 Schematic - add Components (similar to v1.5) - add Pixelix Logo in header
Parts:
- C1, C3, C4: value (none) -> 100n; footprint (none) -> Capacitor_SMD:C_1206_3216Metric_Pad1.33x1.80mm_HandSolder; Manufacturer (none) -> KEMET; Part-No. (none) -> X7R1206B100N
- C2: value (none) -> 1000u / 16V; footprint (none) -> Capacitor_THT:CP_Radial_D8.0mm_P3.50mm; Manufacturer (none) -> Panasonic; Part-No. (none) -> EEU-FR1C102L
- D1: value (none) -> CDSOD323-T05C; footprint (none) -> footprints:CDSOD323-T05C; Part-No. (none) -> CDSOD323-T05C
- F1: value (none) -> 4A; footprint (none) -> footprints:FUSE_0154004.DR; Manufacturer (none) -> Littlefuse; Part-No. (none) -> 0154004.DRT
- J1, J2, J4, J6, J8: value (none) -> Conn_01x02; footprint (none) -> footprints:66200211022; Manufacturer (none) -> Würth Elektronik; Part-No. (none) -> 66200211022
- J3, J7: value (none) -> Conn_01x03; footprint (none) -> footprints:66200311022; Manufacturer (none) -> Würth Elektronik; Part-No. (none) -> 66200311022
- J5: value (none) -> Conn_02x05_Odd_Even; footprint (none) -> footprints:61201021621; Manufacturer (none) -> Würth Elektronik; Part-No. (none) -> 61201021621
- Q1: value (none) -> NMOS_GSD_BSS138; footprint (none) -> Package_TO_SOT_SMD:SOT-23_Handsoldering; Manufacturer (none) -> Onsemi; Part-No. (none) -> BSS138
- Q2: value (none) -> PMOS_GDS_STD26P3LLH6; footprint (none) -> Package_TO_SOT_SMD:TO-252-3_TabPin2; Manufacturer (none) -> STMicroelectronics; Part-No. (none) -> STD26P3LLH6
- R1: value (none) -> 10k; footprint (none) -> Resistor_SMD:R_1206_3216Metric_Pad1.30x1.75mm_HandSolder; Manufacturer (none) -> Yageo; Part-No. (none) -> RC1206JR-0710KL
- R2: value (none) -> 1k; footprint (none) -> Resistor_SMD:R_1206_3216Metric_Pad1.30x1.75mm_HandSolder; Manufacturer (none) -> YAGEO; Part-No. (none) -> RC1206JR-071KL
- R3: value (none) -> 1.2k; footprint (none) -> Resistor_SMD:R_1206_3216Metric_Pad1.30x1.75mm_HandSolder; Manufacturer (none) -> YAGEO; Part-No. (none) -> RC1206JR-071K2L
- R4: value (none) -> 100k; footprint (none) -> Resistor_SMD:R_1206_3216Metric_Pad1.30x1.75mm_HandSolder; Manufacturer (none) -> KOA; Part-No. (none) -> RK73H2BTTD14
- R5, R6, R7, R8: value (none) -> 100; footprint (none) -> Resistor_SMD:R_1206_3216Metric_Pad1.30x1.75mm_HandSolder; Manufacturer (none) -> YAGEO; Part-No. (none) -> RC1206JR-07100RL

Commit message: Board v2.0 Schematic - add Mounting Holes - some small fixes
Parts:
- added H1, H2, H3, H4: MountingHole_Pad, MountingHole:MountingHole_2.2mm_M2_Pad_Via, symbol Mechanical:MountingHole_Pad
Connections:
- no-connect marks 1 -> 5
Other:
- note added: "Mounting Holes"
Changed lines of the file:
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@@
   (junction (at 210.82 152.4) (diameter 0) (color 0 0 0 0)
   )
+  (no_connect (at 180.34 162.56))
+  (no_connect (at 189.23 153.67))
+  (no_connect (at 180.34 153.67))
+  (no_connect (at 189.23 162.56))
   (no_connect (at 229.87 152.4))
   (wire (pts (xy 111.76 101.6) (xy 111.76 99.06))
@@
     (stroke (width 0) (type default) (color 0 0 0 0))
   )
+  (polyline (pts (xy 195.58 163.83) (xy 195.58 147.32))
+    (stroke (width 0) (type default) (color 0 0 0 0))
+  )
   (wire (pts (xy 127 52.07) (xy 90.17 52.07))
     (stroke (width 0) (type default) (color 0 0 0 0))
@@
     (stroke (width 0) (type default) (color 0 0 0 0))
   )
+  (polyline (pts (xy 177.8 163.83) (xy 195.58 163.83))
+    (stroke (width 0) (type default) (color 0 0 0 0))
+  )
   (wire (pts (xy 252.73 106.68) (xy 252.73 113.03))
     (stroke (width 0) (type default) (color 0 0 0 0))
@@
     (stroke (width 0) (type default) (color 0 0 0 0))
   )
+  (polyline (pts (xy 177.8 147.32) (xy 177.8 163.83))
+    (stroke (width 0) (type default) (color 0 0 0 0))
+  )
   (wire (pts (xy 182.88 104.14) (xy 182.88 97.79))
     (stroke (width 0) (type default) (color 0 0 0 0))
@@
   )
   (wire (pts (xy 60.96 175.26) (xy 60.96 179.07))
+    (stroke (width 0) (type default) (color 0 0 0 0))
+  )
+  (polyline (pts (xy 177.8 147.32) (xy 195.58 147.32))
     (stroke (width 0) (type default) (color 0 0 0 0))
   )
@@
     (effects (font (size 1.27 1.27)) (justify left bottom))
   )
+  (text "Mounting Holes" (at 177.8 146.05 0)
+    (effects (font (size 1.27 1.27)) (justify left bottom))
+  )
   (text "Input: 5 V / max. 4 A" (at 17.78 143.51 0)
     (effects (font (size 1.27 1.27) italic) (justify left bottom))
@@
     (pin "3")
   )
+  (symbol (lib_id "Mechanical:MountingHole_Pad") (at 189.23 151.13 0) (unit 1)
+    (in_bom yes) (on_board yes) (fields_autoplaced)
+    (property "Reference" "H3" (id 0) (at 191.77 149.8599 0)
+      (effects (font (size 1.27 1.27)) (justify left))
+    )
+    (property "Value" "MountingHole_Pad" (id 1) (at 191.77 151.1299 0)
+      (effects (font (size 1.27 1.27)) (justify left) hide)
+    )
+    (property "Footprint" "MountingHole:MountingHole_2.2mm_M2_Pad_Via" (id 2) (at 189.23 151.13 0)
+      (effects (font (size 1.27 1.27)) hide)
+    )
+    (property "Datasheet" "~" (id 3) (at 189.23 151.13 0)
+      (effects (font (size 1.27 1.27)) hide)
+    )
+    (pin "1")
+  )
+  (symbol (lib_id "Mechanical:MountingHole_Pad") (at 189.23 160.02 0) (unit 1)
+    (in_bom yes) (on_board yes) (fields_autoplaced)
+    (property "Reference" "H4" (id 0) (at 191.77 158.7499 0)
+      (effects (font (size 1.27 1.27)) (justify left))
+    )
+    (property "Value" "MountingHole_Pad" (id 1) (at 191.77 160.0199 0)
+      (effects (font (size 1.27 1.27)) (justify left) hide)
+    )
+    (property "Footprint" "MountingHole:MountingHole_2.2mm_M2_Pad_Via" (id 2) (at 189.23 160.02 0)
+      (effects (font (size 1.27 1.27)) hide)
+    )
+    (property "Datasheet" "~" (id 3) (at 189.23 160.02 0)
+      (effects (font (size 1.27 1.27)) hide)
+    )
+    (pin "1")
+  )
+  (symbol (lib_id "Mechanical:MountingHole_Pad") (at 180.34 160.02 0) (unit 1)
+    (in_bom yes) (on_board yes) (fields_autoplaced)
+    (property "Reference" "H2" (id 0) (at 182.88 158.7499 0)
+      (effects (font (size 1.27 1.27)) (justify left))
+    )
+    (property "Value" "MountingHole_Pad" (id 1) (at 182.88 160.0199 0)
+      (effects (font (size 1.27 1.27)) (justify left) hide)
+    )
+    (property "Footprint" "MountingHole:MountingHole_2.2mm_M2_Pad_Via" (id 2) (at 180.34 160.02 0)
+      (effects (font (size 1.27 1.27)) hide)
+    )
+    (property "Datasheet" "~" (id 3) (at 180.34 160.02 0)
+      (effects (font (size 1.27 1.27)) hide)
+    )
+    (pin "1")
+  )
+  (symbol (lib_id "Mechanical:MountingHole_Pad") (at 180.34 151.13 0) (unit 1)
+    (in_bom yes) (on_board yes) (fields_autoplaced)
+    (property "Reference" "H1" (id 0) (at 182.88 149.8599 0)
+      (effects (font (size 1.27 1.27)) (justify left))
+    )
+    (property "Value" "MountingHole_Pad" (id 1) (at 182.88 151.1299 0)
+      (effects (font (size 1.27 1.27)) (justify left) hide)
+    )
+    (property "Footprint" "MountingHole:MountingHole_2.2mm_M2_Pad_Via" (id 2) (at 180.34 151.13 0)
+      (effects (font (size 1.27 1.27)) hide)
+    )
+    (property "Datasheet" "~" (id 3) (at 180.34 151.13 0)
+      (effects (font (size 1.27 1.27)) hide)
+    )
+    (pin "1")
+  )
   (sheet (at 127 25.4) (size 38.1 45.72) (fields_autoplaced)
     (stroke (width 0) (type solid) (color 0 0 0 0))
@@
       (reference "F1") (unit 1) (value "4A") (footprint "footprints:FUSE_0154004.DR")
     )
+    (path "/fd185309-3459-4e5b-93ce-02f4de15388f"
+      (reference "H1") (unit 1) (value "MountingHole_Pad") (footprint "MountingHole:MountingHole_2.2mm_M2_Pad_Via")
+    )
+    (path "/f492d757-a7bf-40b4-b989-2f36c88548d8"
+      (reference "H2") (unit 1) (value "MountingHole_Pad") (footprint "MountingHole:MountingHole_2.2mm_M2_Pad_Via")
+    )
+    (path "/8f12766a-e3ab-45e4-87ca-e76de44f5e1c"
+      (reference "H3") (unit 1) (value "MountingHole_Pad") (footprint "MountingHole:MountingHole_2.2mm_M2_Pad_Via")
+    )
+    (path "/e3b3e1bb-fe61-4e34-84a5-afbefa9c2396"
+      (reference "H4") (unit 1) (value "MountingHole_Pad") (footprint "MountingHole:MountingHole_2.2mm_M2_Pad_Via")
+    )
     (path "/00000000-0000-0000-0000-000062329096"

Commit message: Board v2.0 PCB - rotate C2 (1000u Elko) - create new step file
Parts:
- C2: footprint Capacitor_THT:CP_Radial_D8.0mm_P3.50mm -> footprints:CP_Radial_D8.0mm_P3.50mm_horizontal
Changed lines of the file:
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@@
   (title_block
     (title "Pixelix")
-    (date "2022-08-12")
+    (date "2022-09-05")
     (rev "2.0")
     (comment 1 "Schneider, Niklas")
@@
       (effects (font (size 1.27 1.27)) (justify left))
     )
-    (property "Footprint" "Capacitor_THT:CP_Radial_D8.0mm_P3.50mm" (id 2) (at 119.0752 171.45 0)
+    (property "Footprint" "footprints:CP_Radial_D8.0mm_P3.50mm_horizontal" (id 2) (at 119.0752 171.45 0)
       (effects (font (size 1.27 1.27)) hide)
     )
@@
     )
     (path "/00000000-0000-0000-0000-000062526401"
-      (reference "C2") (unit 1) (value "1000u / 16V") (footprint "Capacitor_THT:CP_Radial_D8.0mm_P3.50mm")
+      (reference "C2") (unit 1) (value "1000u / 16V") (footprint "footprints:CP_Radial_D8.0mm_P3.50mm_horizontal")
     )
     (path "/00000000-0000-0000-0000-0000625128b9"

Commit message: Board v2.0 PCB - finished Version 2.0 with the ordering of PCBs and components
Parts:
- H1, H2, H3, H4: Manufacturer (none) -> -; Part-No. (none) -> -
Changed lines of the file:
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@@
   (title_block
     (title "Pixelix")
-    (date "2022-09-12")
+    (date "2022-09-14")
     (rev "2.0")
     (comment 1 "Schneider, Niklas")
@@
       (effects (font (size 1.27 1.27)) hide)
     )
+    (property "Manufacturer" "-" (id 4) (at 189.23 151.13 0)
+      (effects (font (size 1.27 1.27)) hide)
+    )
+    (property "Part-No." "-" (id 5) (at 189.23 151.13 0)
+      (effects (font (size 1.27 1.27)) hide)
+    )
     (pin "1")
   )
@@
       (effects (font (size 1.27 1.27)) hide)
     )
+    (property "Manufacturer" "-" (id 4) (at 189.23 160.02 0)
+      (effects (font (size 1.27 1.27)) hide)
+    )
+    (property "Part-No." "-" (id 5) (at 189.23 160.02 0)
+      (effects (font (size 1.27 1.27)) hide)
+    )
     (pin "1")
   )
@@
       (effects (font (size 1.27 1.27)) hide)
     )
+    (property "Manufacturer" "-" (id 4) (at 180.34 160.02 0)
+      (effects (font (size 1.27 1.27)) hide)
+    )
+    (property "Part-No." "-" (id 5) (at 180.34 160.02 0)
+      (effects (font (size 1.27 1.27)) hide)
+    )
     (pin "1")
   )
@@
       (effects (font (size 1.27 1.27)) hide)
     )
+    (property "Manufacturer" "-" (id 4) (at 180.34 151.13 0)
+      (effects (font (size 1.27 1.27)) hide)
+    )
+    (property "Part-No." "-" (id 5) (at 180.34 151.13 0)
+      (effects (font (size 1.27 1.27)) hide)
+    )
