File: doc/boards/pixelix/v2.1/Pixelix.kicad_pcb (KiCad board)
At the start: 2 copper layers, 100 x 50 mm, 31 parts, among them J1 Conn_01x02, J2 Conn_01x02, J3 Conn_01x03, J4 Conn_01x02, J5 Conn_02x05_Odd_Even, J6 Conn_01x02, J7 Conn_01x03, J8 Conn_01x02, Q1 NMOS_GSD_BSS138, Q2 PMOS_GDS_STD26P3LLH6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

Commit message: #91 HW v2.1: - One Wire added (see #40) - 3V3 and GND to I2S, I2C and One-Wire interface added - Testpoint added
Parts:
- added J9: Conn_01x02, footprints:66200211022, F.Cu at (126.4, 74.7)
- added TP1: TestPoint, Connector_PinHeader_2.54mm:PinHeader_1x01_P2.54mm_Vertical, F.Cu at (138.6, 88.0)
- J3, J7: value Conn_01x03 -> Conn_02x02; footprint footprints:66200311022 -> footprints:66200421022
- J4: value Conn_01x02 -> Conn_02x02; footprint footprints:66200211022 -> footprints:66200421022
- J5: value Conn_02x05_Odd_Even -> Conn_01x02; footprint footprints:61201021621 -> footprints:66200211022
- J6: value Conn_01x02 -> Conn_02x05_Odd_Even; footprint footprints:66200211022 -> footprints:61201021621
- J8: value Conn_01x02 -> Conn_02x03; footprint footprints:66200211022 -> footprints:66200621022
- moved J5 64.1 mm to (105.6, 87.4), turned to -90 degrees
- moved J6 62.8 mm to (168.4, 74.7), turned to 180 degrees
- moved R2 59.3 mm to (193.9, 81.5), turned to 0 degrees
- moved J1 56.2 mm to (193.8, 74.7)
- moved G*** 46.8 mm to (142.5, 98.0), turned to 90 degrees
- moved J7 44.7 mm to (105.6, 75.0), turned to -90 degrees
- moved J3 41.7 mm to (137.6, 74.7), turned to 180 degrees
- moved J8 24.0 mm to (150.4, 74.7)
- moved J4 14.0 mm to (105.6, 101.4)
- moved C4 3.03 mm to (126.4, 81.7)
- moved R3 1.55 mm to (125.0, 90.9)
- moved Q2 0.84 mm to (132.8, 100.8)
- turned C3 to -90 degrees
Connections:
- A1 pad 11: unconnected-(A1-Pad11) -> /ONE-Wire_DHT_IN
- A1 pad 20: unconnected-(A1-Pad20) -> /TEST_Pin
- A1 pad 5: unconnected-(A1-Pad5) -> /I2S_CLK
- A1 pad 6: unconnected-(A1-Pad6) -> /I2S_WS
- A1 pad 8: /I2S_WS -> unconnected-(A1-I39/A3-Pad8)
- A1 pad 9: /I2S_CLK -> unconnected-(A1-IO36/A4-Pad9)
- J3 pad 2: /VCC-PROTECTED -> GND
- J3 pad 3: /HV-DATA-OUT -> /ONE-Wire_DHT_IN
- J4 pad 1: /USER-BUTTON -> GND
- J5 pad 1: +3V3 -> GND
- J5 pad 2: Net-(J5-Pad2) -> /USER-BUTTON
- J6 pad 1: /SCL -> +3V3
- J6 pad 2: /SDA -> Net-(J6-Pin_2)
- J7 pad 1: /I2S_CLK -> GND
- J7 pad 2: /I2S_WS -> /SCL
- J7 pad 3: /I2S_Data_IN -> /SDA
- J8 pad 1: /RESET -> GND
- R5 pad 1: Net-(J5-Pad2) -> Net-(J6-Pin_2)
- R6 pad 1: Net-(J5-Pad4) -> Net-(J6-Pin_4)
- R7 pad 1: Net-(J5-Pad6) -> Net-(J6-Pin_6)
- R8 pad 1: Net-(J5-Pad8) -> Net-(J6-Pin_8)
- U1 pad 23: unconnected-(U1-Pad23) -> /TEST_Pin
- U1 pad 29: unconnected-(U1-Pad29) -> /ONE-Wire_DHT_IN
Routing:
- net /TEST_Pin: track 0.00 -> 48.6 mm, vias 0 -> 1
- net /ONE-Wire_DHT_IN: track 0.00 -> 46.0 mm, vias 0 -> 1
- net +3V3: track 106.7 -> 145.4 mm
- net /LDR-ANALOG-IN: track 70.8 -> 48.6 mm, vias 1 -> 2
- net /I2S_WS: track 55.0 -> 64.6 mm, vias 1 -> 0
- net /I2S_CLK: track 57.6 -> 64.7 mm, vias 0 -> 1
- net /SDA: track 94.3 -> 89.9 mm
- net /HV-DATA-OUT: track 19.5 -> 16.5 mm
- net Net-(J6-Pin_2): track 0.00 -> 2.48 mm
- net Net-(J5-Pad2): track 2.48 -> 0.00 mm
- net Net-(J6-Pin_4): track 0.00 -> 2.48 mm
- net Net-(J5-Pad4): track 2.48 -> 0.00 mm
- net Net-(J6-Pin_6): track 0.00 -> 2.48 mm
- net Net-(J5-Pad6): track 2.48 -> 0.00 mm
- net Net-(J6-Pin_8): track 0.00 -> 2.48 mm
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Other:
- board text added: "One-Wire"
- board text added: "V2.1"
- board text removed: "V2.0"
